Commit message: testing

File: robot.urdf (robot description, URDF)
Before this commit: robot static, 31 links, 30 joints
Links:
- removed link ebox
Joints:
- removed joint ebox_to_cam
- removed joint table_to_ebox
- added joint world_to_cam: type fixed, parent world, child center_cam, origin xyz=0.365 0.85 0.75 rpy=1.57 0.0 3.14
