Commit message: template fixed

File: examples/workcell.template.urdf (robot description, URDF)
Before this commit: robot static, 30 links, 29 joints
Links:
- link center_cam_link: geometry collision box size=0.026 0.124 0.029; visual mesh filename={SIMS_CORE}/examples/meshes/camera/d455.stl scale=0.001 0.001 0.001
- link left_base_link: geometry collision mesh filename={SIMS_CORE}/examples/meshes/piper/base_link.STL; visual mesh filename={SIMS_CORE}/examples/meshes/piper/base_link.dae
- link left_cam_link: geometry collision box size=0.023 0.042 0.042; visual mesh filename={SIMS_CORE}/examples/meshes/camera/d405.stl scale=0.001 0.001 0.001
- link left_link1: geometry collision mesh filename={SIMS_CORE}/examples/meshes/piper/link1.STL; visual mesh filename={SIMS_CORE}/examples/meshes/piper/link1.dae
- link left_link2: geometry collision mesh filename={SIMS_CORE}/examples/meshes/piper/link2.STL; visual mesh filename={SIMS_CORE}/examples/meshes/piper/link2.dae
- link left_link3: geometry collision mesh filename={SIMS_CORE}/examples/meshes/piper/link3.STL; visual mesh filename={SIMS_CORE}/examples/meshes/piper/link3.dae
- link left_link4: geometry collision mesh filename={SIMS_CORE}/examples/meshes/piper/link4.STL; visual mesh filename={SIMS_CORE}/examples/meshes/piper/link4.dae
- link left_link5: geometry collision mesh filename={SIMS_CORE}/examples/meshes/piper/link5.STL; visual mesh filename={SIMS_CORE}/examples/meshes/piper/link5.dae
- link left_link6: geometry collision mesh filename={SIMS_CORE}/examples/meshes/piper/link6_1.STL; visual mesh filename={SIMS_CORE}/examples/meshes/piper/link6.dae
- link left_link7.1: geometry collision mesh filename={SIMS_CORE}/examples/meshes/piper/link7.STL; visual mesh filename={SIMS_CORE}/examples/meshes/piper/link7.dae
- link left_link7.2: geometry collision mesh filename={SIMS_CORE}/examples/meshes/piper/link8.STL; visual mesh filename={SIMS_CORE}/examples/meshes/piper/link8.dae
- link right_base_link: geometry collision mesh filename={SIMS_CORE}/examples/meshes/piper/base_link.STL; visual mesh filename={SIMS_CORE}/examples/meshes/piper/base_link.dae
- link right_cam_link: geometry collision box size=0.023 0.042 0.042; visual mesh filename={SIMS_CORE}/examples/meshes/camera/d405.stl scale=0.001 0.001 0.001
- link right_link1: geometry collision mesh filename={SIMS_CORE}/examples/meshes/piper/link1.STL; visual mesh filename={SIMS_CORE}/examples/meshes/piper/link1.dae
- link right_link2: geometry collision mesh filename={SIMS_CORE}/examples/meshes/piper/link2.STL; visual mesh filename={SIMS_CORE}/examples/meshes/piper/link2.dae
- link right_link3: geometry collision mesh filename={SIMS_CORE}/examples/meshes/piper/link3.STL; visual mesh filename={SIMS_CORE}/examples/meshes/piper/link3.dae
- link right_link4: geometry collision mesh filename={SIMS_CORE}/examples/meshes/piper/link4.STL; visual mesh filename={SIMS_CORE}/examples/meshes/piper/link4.dae
- link right_link5: geometry collision mesh filename={SIMS_CORE}/examples/meshes/piper/link5.STL; visual mesh filename={SIMS_CORE}/examples/meshes/piper/link5.dae
- link right_link6: geometry collision mesh filename={SIMS_CORE}/examples/meshes/piper/link6_1.STL; visual mesh filename={SIMS_CORE}/examples/meshes/piper/link6.dae
- link right_link7.1: geometry collision mesh filename={SIMS_CORE}/examples/meshes/piper/link7.STL; visual mesh filename={SIMS_CORE}/examples/meshes/piper/link7.dae
- link right_link7.2: geometry collision mesh filename={SIMS_CORE}/examples/meshes/piper/link8.STL; visual mesh filename={SIMS_CORE}/examples/meshes/piper/link8.dae
- link table_corner: geometry collision mesh filename={SIMS_CORE}/examples/meshes/workcell/table.STL scale=0.001 0.001 0.001; visual mesh filename={SIMS_CORE}/examples/meshes/workcell/table.STL scale=0.001 0.001 0.001
